File: TD-XPAH_hAT.kicad_pcb (KiCad board)
At the start: 2 copper layers, 47.1 x 50 mm, 6 parts, among them J1 Conn_01x14_Male, J2 Conn_01x12_Male, J3 Conn_01x14_Male

Commit message: rename to TD-XPAH
Parts:
- moved G*** 29.9 mm to (208.9, 102.4), turned to 90 degrees
Changed lines of the file:
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@@
     (descr "Through hole straight pin header, 1x14, 2.54mm pitch, single row")
     (tags "Through hole pin header THT 1x14 2.54mm single row")
-    (property "Sheetfile" "TD-XPAH01_hAT.kicad_sch")
+    (property "Sheetfile" "TD-XPAH_hAT.kicad_sch")
     (property "Sheetname" "")
     (attr through_hole)
@@
     (descr "Mounting Hole 3.2mm, M3")
     (tags "mounting hole 3.2mm m3")
-    (property "Sheetfile" "TD-XPAH01_hAT.kicad_sch")
+    (property "Sheetfile" "TD-XPAH_hAT.kicad_sch")
     (property "Sheetname" "")
     (attr exclude_from_pos_files)
@@
     (descr "Mounting Hole 3.2mm, M3")
     (tags "mounting hole 3.2mm m3")
-    (property "Sheetfile" "TD-XPAH01_hAT.kicad_sch")
+    (property "Sheetfile" "TD-XPAH_hAT.kicad_sch")
     (property "Sheetname" "")
     (attr exclude_from_pos_files)
@@
     (descr "Through hole straight pin header, 1x12, 2.54mm pitch, single row")
     (tags "Through hole pin header THT 1x12 2.54mm single row")
-    (property "Sheetfile" "TD-XPAH01_hAT.kicad_sch")
+    (property "Sheetfile" "TD-XPAH_hAT.kicad_sch")
     (property "Sheetname" "")
     (attr through_hole)
@@
     (descr "Through hole straight pin header, 1x14, 2.54mm pitch, single row")
     (tags "Through hole pin header THT 1x14 2.54mm single row")
-    (property "Sheetfile" "TD-XPAH01_hAT.kicad_sch")
+    (property "Sheetfile" "TD-XPAH_hAT.kicad_sch")
     (property "Sheetname" "")
     (attr through_hole)
@@
   )
   (footprint "teledatics:teledatics_logo_kicad_footprint" (layer "F.Cu")
-    (at 178.963547 102.756718 -90)
+    (at 208.864169 102.373282 90)
     (attr board_only exclude_from_pos_files exclude_from_bom)
     (fp_text reference "G***" (at 0 0 90) (layer "F.Fab")
